File: pcb.brd (EAGLE design)
At the start: 57.1 x 33 mm, 13 parts, among them J1 455-1750-1-ND, J2 AUDIO_JACK_TRRSSMD_RA, U1 ESP-WROVER-32ESP-WROVER-32, X1 MAB5SH

Commit message: small fixes
Parts:
- IC1: value (none) -> MCP1826S33
Connections:
- net CLOCK: now also J3.A7, J3.B7, U1.P$10; no longer J3.A6, J3.B6, U1.P$11
- net START: now also J3.A6, J3.B6, U1.P$11; no longer J3.A7, J3.B7, U1.P$10
Changed lines of the file:
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@@
 <attribute name="SF_ID" value="PRT-12639" x="58.42" y="7.62" size="1.778" layer="27" rot="R180" display="off"/>
 </element>
-<element name="IC1" library="linear-technology" package="SOT223" value="" x="7.62" y="24.13" rot="R90">
+<element name="IC1" library="linear-technology" package="SOT223" value="MCP1826S33" x="7.62" y="24.13" rot="R90">
 <attribute name="MPN" value="LT1129CST-5#PBF" x="7.62" y="24.13" size="1.778" layer="27" rot="R90" display="off"/>
 <attribute name="OC_FARNELL" value="1663375" x="7.62" y="24.13" size="1.778" layer="27" rot="R90" display="off"/>
@@
 <wire x1="36.83" y1="17.78" x2="38.42" y2="17.78" width="0.254" layer="1"/>
 </signal>
-<signal name="START">
+<signal name="CLOCK">
 <contactref element="U1" pad="P$10"/>
 <wire x1="16.76" y1="15.42" x2="12.7" y2="15.42" width="0.254" layer="1"/>
@@
 <wire x1="7.28" y1="13.72" x2="6.35" y2="13.72" width="0.254" layer="1"/>
 </signal>
-<signal name="CLOCK">
+<signal name="START">
 <contactref element="U1" pad="P$11"/>
 <wire x1="11.86" y1="14.15" x2="16.76" y2="14.15" width="0.254" layer="1"/>
